Commit message: Update code (AAAI-26 Main Conference)

File: Agent/assets/ball.urdf (robot description, URDF)
Before this commit: robot ball, 1 links, 0 joints
Links:
- link ball: mass 0.0005 -> 0.05

File: Agent/assets/no_mass_ball.urdf (robot description, URDF)
Before this commit: robot ball, 1 links, 0 joints
Links:
- link ball: geometry collision sphere radius=0.02; visual sphere radius=0.02

File: Agent/assets/pendulum.urdf (robot description, URDF)
Before this commit: robot pendulum, 7 links, 6 joints
Links:
- link hook1: mass 5000 -> 0.00001
- link hook2: mass 5000 -> 0.00001
- link hook3: mass 5000 -> 0.00001
- link rod: mass 0.01 -> 0.00000001
- link top: mass 5000 -> 0.000001
